Commit message: Add dynamic obstacle tracking and collision.

File: src/gazebo/launch/env.urdf (robot description, URDF)
Before this commit: robot environment, 12 links, 11 joints
Links:
- added link moving_obstacle_bottom/body; visual box size=1 1 1.5
- added link moving_obstacle_top/body; visual box size=1 1 1.5
